File: Feather-SAM-M8Q-GPS.sch (KiCad schematic (older format))
At the start: 33 parts, among them U1 ublox_SAM-M8Q

Commit message: Rev1.5 of SAM-M8Q GPS
Parts:
- added JP10, JP11, JP12, JP9: ~, Jumper:SolderJumper-2_P1.3mm_Open_RoundedPad1.0x1.5mm, symbol Jumper:SolderJumper_2_Open
- RX1, RX2, RX3, TX1, TX2, TX3, TX4: footprint Connector_Pin:Pin_D1.0mm_L10.0mm -> ~Connector_Pin:Pin_D1.0mm_L10.0mm
Connections:
- net 10`: now also JP10.1 (A)
- net 11`: now also JP9.2 (B)
- net 12: now also JP12.1 (A)
- net 9`: now also JP11.1 (A)
- net INT: now also JP10.2 (B)
- net PPS: now also JP12.2 (B)
- net SCL2: no longer JP8.1 (A), R2.1, R9.2
- net SDA2: no longer JP7.1 (A), R1.1, R8.2
- net ~RESET: now also JP11.2 (B)
- net ~SAFE: now also JP9.1 (A)
- new net: JP8.1 (A), R2.1, R9.2
- new net: JP7.1 (A), R1.1, R8.2
Changed lines of the file:
@@
 F 0 "TX1" H 9630 1742 50  0000 L CNN
 F 1 "TX" H 9630 1651 50  0000 L CNN
-F 2 "Connector_Pin:Pin_D1.0mm_L10.0mm" H 9550 1700 50  0001 C CNN
+F 2 "~Connector_Pin:Pin_D1.0mm_L10.0mm" H 9550 1700 50  0001 C CNN
 F 3 "~" H 9550 1700 50  0001 C CNN
 	1    9550 1700
@@
 F 0 "RX1" H 9630 1942 50  0000 L CNN
 F 1 "RX" H 9630 1851 50  0000 L CNN
-F 2 "Connector_Pin:Pin_D1.0mm_L10.0mm" H 9550 1900 50  0001 C CNN
+F 2 "~Connector_Pin:Pin_D1.0mm_L10.0mm" H 9550 1900 50  0001 C CNN
 F 3 "~" H 9550 1900 50  0001 C CNN
 	1    9550 1900
@@
 Wire Wire Line
 	9150 2350 9250 2350
-Text Label 8650 2250 0    50   ~ 0
-SDA2
-Text Label 8650 2350 0    50   ~ 0
-SCL2
 $Comp
 L Connector_Generic:Conn_01x01 TX2
@@
 F 0 "TX2" H 9680 2842 50  0000 L CNN
 F 1 "SDA" H 9680 2751 50  0000 L CNN
-F 2 "Connector_Pin:Pin_D1.0mm_L10.0mm" H 9600 2800 50  0001 C CNN
+F 2 "~Connector_Pin:Pin_D1.0mm_L10.0mm" H 9600 2800 50  0001 C CNN
 F 3 "~" H 9600 2800 50  0001 C CNN
 	1    9600 2800
@@
 F 0 "RX2" H 9680 3042 50  0000 L CNN
 F 1 "SCL" H 9680 2951 50  0000 L CNN
-F 2 "Connector_Pin:Pin_D1.0mm_L10.0mm" H 9600 3000 50  0001 C CNN
+F 2 "~Connector_Pin:Pin_D1.0mm_L10.0mm" H 9600 3000 50  0001 C CNN
 F 3 "~" H 9600 3000 50  0001 C CNN
 	1    9600 3000
@@
 F 0 "RX3" H 9680 3792 50  0000 L CNN
 F 1 "INT" H 9680 3701 50  0000 L CNN
-F 2 "Connector_Pin:Pin_D1.0mm_L10.0mm" H 9600 3750 50  0001 C CNN
+F 2 "~Connector_Pin:Pin_D1.0mm_L10.0mm" H 9600 3750 50  0001 C CNN
 F 3 "~" H 9600 3750 50  0001 C CNN
 	1    9600 3750
@@
 F 0 "TX4" H 9680 3992 50  0000 L CNN
 F 1 "~RST" H 9680 3901 50  0000 L CNN
-F 2 "Connector_Pin:Pin_D1.0mm_L10.0mm" H 9600 3950 50  0001 C CNN
+F 2 "~Connector_Pin:Pin_D1.0mm_L10.0mm" H 9600 3950 50  0001 C CNN
 F 3 "~" H 9600 3950 50  0001 C CNN
 	1    9600 3950
@@
 F 0 "TX3" H 9680 3592 50  0000 L CNN
 F 1 "~SAFE" H 9680 3501 50  0000 L CNN
-F 2 "Connector_Pin:Pin_D1.0mm_L10.0mm" H 9600 3550 50  0001 C CNN
+F 2 "~Connector_Pin:Pin_D1.0mm_L10.0mm" H 9600 3550 50  0001 C CNN
 F 3 "~" H 9600 3550 50  0001 C CNN
 	1    9600 3550
 	1    0    0    -1
 $EndComp
+Text Label 7000 4800 2    50   ~ 0
+~SAFE
+Text Label 7000 4950 2    50   ~ 0
+INT
+Text Label 6950 5100 2    50   ~ 0
+~RESET
+Text Label 6950 5250 2    50   ~ 0
+PPS
+Wire Wire Line
+	7000 4800 7150 4800
+Wire Wire Line
+	7000 4950 7150 4950
+Wire Wire Line
+	7150 5100 6950 5100
+Wire Wire Line
+	6950 5250 7150 5250
+Text Label 7650 4950 0    50   ~ 0
+10`
+Wire Wire Line
+	7650 4950 7450 4950
+Text Label 7650 5100 0    50   ~ 0
+9`
+Wire Wire Line
+	7650 5100 7450 5100
+Text Label 7650 5250 0    50   ~ 0
+12
+Text Label 7650 4800 0    50   ~ 0
+11`
+Wire Wire Line
+	7650 4800 7450 4800
+Wire Wire Line
+	7450 5250 7650 5250
+$Comp
+L Jumper:SolderJumper_2_Open JP12
+U 1 1 5E2E79E5
+P 7300 5250
+F 0 "JP12" H 7050 5200 50  0000 L CNN
+F 1 "~" V 7345 5318 50  0000 L CNN
+F 2 "Jumper:SolderJumper-2_P1.3mm_Open_RoundedPad1.0x1.5mm" H 7300 5250 50  0001 C CNN
+F 3 "~" H 7300 5250 50  0001 C CNN
+	1    7300 5250
+	-1   0    0    1
+$EndComp
+$Comp
+L Jumper:SolderJumper_2_Open JP11
+U 1 1 5E2E7712
+P 7300 5100
+F 0 "JP11" H 7050 5050 50  0000 L CNN
+F 1 "~" V 7345 5168 50  0000 L CNN
+F 2 "Jumper:SolderJumper-2_P1.3mm_Open_RoundedPad1.0x1.5mm" H 7300 5100 50  0001 C CNN
+F 3 "~" H 7300 5100 50  0001 C CNN
+	1    7300 5100
+	-1   0    0    1
+$EndComp
+$Comp
+L Jumper:SolderJumper_2_Open JP10
+U 1 1 5E2E5126
+P 7300 4950
+F 0 "JP10" H 7050 4900 50  0000 L CNN
+F 1 "~" V 7345 5018 50  0000 L CNN
+F 2 "Jumper:SolderJumper-2_P1.3mm_Open_RoundedPad1.0x1.5mm" H 7300 4950 50  0001 C CNN
+F 3 "~" H 7300 4950 50  0001 C CNN
+	1    7300 4950
+	-1   0    0    1
+$EndComp
+$Comp
+L Jumper:SolderJumper_2_Open JP9
+U 1 1 5E2E4BF9
+P 7300 4800
+F 0 "JP9" H 7400 4850 50  0000 L CNN
+F 1 "~" V 7345 4868 50  0000 L CNN
+F 2 "Jumper:SolderJumper-2_P1.3mm_Open_RoundedPad1.0x1.5mm" H 7300 4800 50  0001 C CNN
+F 3 "~" H 7300 4800 50  0001 C CNN
+	1    7300 4800
+	1    0    0    -1
+$EndComp
